File: EAGLE Schematic/SLB_EXT_EAGLE.brd (EAGLE design)
At the start: 210 x 100 mm, 706 parts, among them J1 16P_HEADER_SMD, J10 DB2EVC-3.81-4P-GN, J11 1803280, J12 KH-PCB-6P6C, J13 WJ15EDGK-3.81-2P, J14 KH-PCB-6P6C, J15 B4B-XH-A(LF)(SN), J17 WJ15EDGK-3.81-2P, J18 B3B-XH-A(LF)(SN), J19 DNI, J2 Phoenix Pluggable 3.81mm 3 way, J20 USB-C-Socket, J21 B3B-XH-A(LF)(SN), J3 Phoenix Pluggable 3.81mm 2 way, J4 B4B-XH-A(LF)(SN), J5 B4B-XH-A(LF)(SN), J6 B4B-XH-A(LF)(SN), J7 B4B-XH-A(LF)(SN), J8 B4B-XH-A(LF)(SN), J9 1803455, K1_TR1 TLP3109A, K1_TR2 TLP3109A, K2 VCF4-1000, P1 DB2EVC-3.81-2P-GN, P10 DB2ERC-5.08-2P-GN, P11 SHROUDED_BOX_HEADER_40, P12 HR911105A, P13 SHROUDED_BOX_HEADER_08, P14 SHROUDED_BOX_HEADER_08, P15 DNI, P16 SHROUDED_BOX_HEADER_08, P17 DB2EVC-3.81-7P-GN, P18_RL1 WJ15EDGK-3.81-2P, P18_RL2 WJ15EDGK-3.81-2P, P19 WJ15EDGK-3.81-2P, P2 DB2EVC-3.81-2P-GN, P20 SHROUDED_BOX_HEADER_08, P21_TR1 WJ15EDGK-3.81-2P, P21_TR2 WJ15EDGK-3.81-2P, P23 22284020, P24 1803329, P25 DNI, P26 DNI, P27 SHROUDED_BOX_HEADER_08, P28 DB2EVC-3.81-2P-GN, P3 DB2EVC-3.81-2P-GN, P4 DB2EVC-3.81-2P-GN, P5 Header 2, P6 WJ15EDGK-3.81-2P, P8 DNI, P9 DNI, Q1 WSF50P10, Q10_RL1 2N7002-7-F, Q10_RL2 2N7002-7-F, Q11 2N7002-7-F, Q12 2N7002-7-F, Q13 ST3422A, Q14 CSD19538Q3A, Q15 CSD19538Q3A, Q16 BSS123, Q17 BSS123, Q2_RL1 ST3422A, Q2_RL2 ST3422A, Q3 2N7002-7-F, Q4 2N7002-7-F, Q5 2N7002-7-F, Q6 2N7002-7-F, Q7 2N7002-7-F, Q8 2N7002-7-F, Q9_TR1 2N7002-7-F, Q9_TR2 2N7002-7-F, U1 SN74AHC1G86DBVR, U10 EL357N-G, U11 W5500, U12 CBMUD1201LAS8, U13 SN75176BDR, U14 ADUM1200ARZ-RL7, U15 EL357N-G, U16 TPS54331DR, U17 STM32F412VGT6STM32F412VGT6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

Commit message: Updated schematic
Connections:
- net HALT_PEN: now also U21.2
- net KPSTR_PEN: now also U22.2
Changed lines of the file:
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@@
 <signal name="HALT_PEN">
 <contactref element="J14" pad="4"/>
+<contactref element="U21" pad="2"/>
+<wire x1="7.773546875" y1="25.77383125" x2="26.824990625" y2="23.701221875" width="0" layer="19" extent="1-1"/>
 </signal>
 <signal name="KPSTR_PEN">
 <contactref element="J14" pad="5"/>
+<contactref element="U22" pad="2"/>
+<wire x1="10.313546875" y1="26.79383125" x2="26.824990625" y2="28.355009375" width="0" layer="19" extent="1-1"/>
 </signal>
 <signal name="N$186">

Commit message: Updated schematic (Incorrectly named NET)
Connections:
- removed net USB_D_R_M: U17.70
- net USB_D_R_N: now also U17.70
Changed lines of the file:
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@@
 <signal name="USB_D_R_N">
 <contactref element="R67" pad="1"/>
+<contactref element="U17" pad="70"/>
+<wire x1="35.036490625" y1="19.8810375" x2="44.499996875" y2="19.991215625" width="0" layer="19" extent="1-1"/>
 </signal>
 <signal name="N$2">
@@
 <wire x1="-10.4" y1="3.378" x2="-12.75" y2="8.5" width="0" layer="19" extent="1-1"/>
 </signal>
-<signal name="USB_D_R_M">
-<contactref element="U17" pad="70"/>
-</signal>
 <signal name="VCAP2">
