File: EAGLE Schematic/SLB_EXT_EAGLE.brd (EAGLE design)
At the start: 210 x 100 mm, 706 parts, among them J1 16P_HEADER_SMD, J10 DB2EVC-3.81-4P-GN, J11 1803280, J12 KH-PCB-6P6C, J13 WJ15EDGK-3.81-2P, J14 KH-PCB-6P6C, J15 B4B-XH-A(LF)(SN), J17 WJ15EDGK-3.81-2P, J18 B3B-XH-A(LF)(SN), J19 DNI, J2 Phoenix Pluggable 3.81mm 3 way, J20 USB-C-Socket, J21 B3B-XH-A(LF)(SN), J3 Phoenix Pluggable 3.81mm 2 way, J4 B4B-XH-A(LF)(SN), J5 B4B-XH-A(LF)(SN), J6 B4B-XH-A(LF)(SN), J7 B4B-XH-A(LF)(SN), J8 B4B-XH-A(LF)(SN), J9 1803455, K1_TR1 TLP3109A, K1_TR2 TLP3109A, K2 VCF4-1000, P1 DB2EVC-3.81-2P-GN, P10 DB2ERC-5.08-2P-GN, P11 SHROUDED_BOX_HEADER_40, P12 HR911105A, P13 SHROUDED_BOX_HEADER_08, P14 SHROUDED_BOX_HEADER_08, P15 DNI, P16 SHROUDED_BOX_HEADER_08, P17 DB2EVC-3.81-7P-GN, P18_RL1 WJ15EDGK-3.81-2P, P18_RL2 WJ15EDGK-3.81-2P, P19 WJ15EDGK-3.81-2P, P2 DB2EVC-3.81-2P-GN, P20 SHROUDED_BOX_HEADER_08, P21_TR1 WJ15EDGK-3.81-2P, P21_TR2 WJ15EDGK-3.81-2P, P23 22284020, P24 1803329, P25 DNI, P26 DNI, P27 SHROUDED_BOX_HEADER_08, P28 DB2EVC-3.81-2P-GN, P3 DB2EVC-3.81-2P-GN, P4 DB2EVC-3.81-2P-GN, P5 Header 2, P6 WJ15EDGK-3.81-2P, P8 DNI, P9 DNI, Q1 WSF50P10, Q10_RL1 2N7002-7-F, Q10_RL2 2N7002-7-F, Q11 2N7002-7-F, Q12 2N7002-7-F, Q13 ST3422A, Q14 CSD19538Q3A, Q15 CSD19538Q3A, Q16 BSS123, Q17 BSS123, Q2_RL1 ST3422A, Q2_RL2 ST3422A, Q3 2N7002-7-F, Q4 2N7002-7-F, Q5 2N7002-7-F, Q6 2N7002-7-F, Q7 2N7002-7-F, Q8 2N7002-7-F, Q9_TR1 2N7002-7-F, Q9_TR2 2N7002-7-F, U1 SN74AHC1G86DBVR, U10 EL357N-G, U11 W5500, U12 CBMUD1201LAS8, U13 SN75176BDR, U14 ADUM1200ARZ-RL7, U15 EL357N-G, U16 TPS54331DR, U17 STM32F412VGT6STM32F412VGT6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

Commit message: Fix disconnected nets on BAT54S components
Connections:
- new net GND\: D53.1
- net GND: now also D35.1, D54.1, D55.1
- net VCC_SYS_5V0: now also D35.2, D53.2, D54.2, D55.2
Changed lines of the file:
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@@
 <wire x1="210" y1="100" x2="210" y2="0" width="0.1524" layer="20"/>
 <wire x1="210" y1="0" x2="0" y2="0" width="0.1524" layer="20"/>
+<dimension x1="0" y1="0" x2="210" y2="0" x3="105" y3="-11.3" textsize="1.778" layer="1"/>
 </plain>
 <attributes>
@@
 <contactref element="C7" pad="2"/>
 <contactref element="L2" pad="1"/>
+<contactref element="D35" pad="1"/>
+<contactref element="D54" pad="1"/>
+<contactref element="D55" pad="1"/>
 <wire x1="197.284796875" y1="55.214596875" x2="199.83645625" y2="55.874996875" width="0" layer="19" extent="1-1"/>
 <wire x1="195.750003125" y1="55.849990625" x2="197.284796875" y2="55.214596875" width="0" layer="19" extent="1-1"/>
@@
 <wire x1="65.6500125" y1="41.875" x2="61.149996875" y2="42.1999875" width="0" layer="19" extent="1-1"/>
 <wire x1="135.1241125" y1="89.875003125" x2="144.16046875" y2="89.875003125" width="0" layer="19" extent="1-1"/>
-<wire x1="65.37829375" y1="71.854625" x2="57.61575625" y2="77.3993375" width="0" layer="19" extent="1-1"/>
-<wire x1="66.929990625" y1="73.0362" x2="65.37829375" y2="71.854625" width="0" layer="19" extent="1-1"/>
-<wire x1="70.739990625" y1="68.0862" x2="66.929990625" y2="73.0362" width="0" layer="19" extent="1-1"/>
-<wire x1="72.249990625" y1="76.62499375" x2="66.929990625" y2="73.0362" width="0" layer="19" extent="1-1"/>
-<wire x1="75.624990625" y1="76.62499375" x2="72.249990625" y2="76.62499375" width="0" layer="19" extent="1-1"/>
-<wire x1="81.46360625" y1="71.854625" x2="75.624990625" y2="76.62499375" width="0" layer="19" extent="1-1"/>
-<wire x1="88.700003125" y1="75.124996875" x2="81.46360625" y2="71.854625" width="0" layer="19" extent="1-1"/>
-<wire x1="97.67365625" y1="71.854625" x2="88.700003125" y2="75.124996875" width="0" layer="19" extent="1-1"/>
+<wire x1="91.099996875" y1="66.800003125" x2="89.179984375" y2="57.64499375" width="0" layer="19" extent="1-1"/>
+<wire x1="91.099996875" y1="70.249984375" x2="91.099996875" y2="66.800003125" width="0" layer="19" extent="1-1"/>
+<wire x1="85.9749875" y1="66.800003125" x2="91.099996875" y2="66.800003125" width="0" layer="19" extent="1-1"/>
+<wire x1="88.700003125" y1="75.124996875" x2="91.099996875" y2="70.249984375" width="0" layer="19" extent="1-1"/>
+<wire x1="97.67365625" y1="71.854625" x2="91.099996875" y2="70.249984375" width="0" layer="19" extent="1-1"/>
 <wire x1="99.430003125" y1="73.0362" x2="97.67365625" y2="71.854625" width="0" layer="19" extent="1-1"/>
 <wire x1="103.240003125" y1="68.0862" x2="99.430003125" y2="73.0362" width="0" layer="19" extent="1-1"/>
 <wire x1="104.750003125" y1="76.62499375" x2="99.430003125" y2="73.0362" width="0" layer="19" extent="1-1"/>
 <wire x1="108.125" y1="76.62499375" x2="104.750003125" y2="76.62499375" width="0" layer="19" extent="1-1"/>
+<wire x1="81.46360625" y1="71.854625" x2="85.9749875" y2="66.800003125" width="0" layer="19" extent="1-1"/>
 <wire x1="113.883709375" y1="71.854625" x2="108.125" y2="76.62499375" width="0" layer="19" extent="1-1"/>
+<wire x1="75.624990625" y1="76.62499375" x2="81.46360625" y2="71.854625" width="0" layer="19" extent="1-1"/>
+<wire x1="72.249990625" y1="76.62499375" x2="75.624990625" y2="76.62499375" width="0" layer="19" extent="1-1"/>
+<wire x1="66.929990625" y1="73.0362" x2="72.249990625" y2="76.62499375" width="0" layer="19" extent="1-1"/>
+<wire x1="65.37829375" y1="71.854625" x2="66.929990625" y2="73.0362" width="0" layer="19" extent="1-1"/>
+<wire x1="70.739990625" y1="68.0862" x2="66.929990625" y2="73.0362" width="0" layer="19" extent="1-1"/>
 <wire x1="130.775003125" y1="81.125009375" x2="135.1241125" y2="89.875003125" width="0" layer="19" extent="1-1"/>
 <wire x1="128.02499375" y1="81.125009375" x2="130.775003125" y2="81.125009375" width="0" layer="19" extent="1-1"/>
@@
 <contactref element="L1" pad="1"/>
 <contactref element="C7" pad="1"/>
+<contactref element="D54" pad="2"/>
+<contactref element="D55" pad="2"/>
+<contactref element="D35" pad="2"/>
+<contactref element="D53" pad="2"/>
 <wire x1="200.35000625" y1="51.624990625" x2="199.83645625" y2="55.224996875" width="0" layer="19" extent="1-1"/>
 <wire x1="201.375009375" y1="50.774990625" x2="200.35000625" y2="51.624990625" width="0" layer="19" extent="1-1"/>
@@
 <wire x1="103.000003125" y1="76.62499375" x2="106.375" y2="76.62499375" width="0" layer="19" extent="1-1"/>
 <wire x1="96.197" y1="61.749990625" x2="105.50498125" y2="61.749990625" width="0" layer="19" extent="1-1"/>
-<wire x1="86.888990625" y1="61.749990625" x2="96.197" y2="61.749990625" width="0" layer="19" extent="1-1"/>
-<wire x1="75.819990625" y1="68.0862" x2="86.888990625" y2="61.749990625" width="0" layer="19" extent="1-1"/>
+<wire x1="91.099996875" y1="68.700003125" x2="96.197" y2="61.749990625" width="0" layer="19" extent="1-1"/>
+<wire x1="91.099996875" y1="72.149984375" x2="91.099996875" y2="68.700003125" width="0" layer="19" extent="1-1"/>
+<wire x1="85.9749875" y1="72.075003125" x2="91.099996875" y2="72.149984375" width="0" layer="19" extent="1-1"/>
+<wire x1="85.300003125" y1="75.124996875" x2="85.9749875" y2="72.075003125" width="0" layer="19" extent="1-1"/>
+<wire x1="85.9749875" y1="68.700003125" x2="85.9749875" y2="72.075003125" width="0" layer="19" extent="1-1"/>
+<wire x1="86.888990625" y1="61.749990625" x2="85.9749875" y2="68.700003125" width="0" layer="19" extent="1-1"/>
+<wire x1="75.819990625" y1="68.0862" x2="85.9749875" y2="68.700003125" width="0" layer="19" extent="1-1"/>
 <wire x1="73.874990625" y1="76.62499375" x2="75.819990625" y2="68.0862" width="0" layer="19" extent="1-1"/>
 <wire x1="70.499990625" y1="76.62499375" x2="73.874990625" y2="76.62499375" width="0" layer="19" extent="1-1"/>
-<wire x1="85.300003125" y1="75.124996875" x2="73.874990625" y2="76.62499375" width="0" layer="19" extent="1-1"/>
 <wire x1="112.500003125" y1="88.12499375" x2="106.375" y2="76.62499375" width="0" layer="19" extent="1-1"/>
 <wire x1="80.16666875" y1="88.12499375" x2="73.874990625" y2="76.62499375" width="0" layer="19" extent="1-1"/>
@@
 <wire x1="43.13" y1="41.99999375" x2="39.499996875" y2="52.375003125" width="0" layer="19" extent="1-1"/>
 </signal>
+<signal name="GND\">
+<contactref element="D53" pad="1"/>
+</signal>
 </signals>
